Commit message: Updates to allow checkerboard motion to be correctly simulated

File: med7pf_description/urdf/med7pf.urdf.xacro (robot description, xacro)
@@ -20,5 +20,5 @@
     </xacro:med7>
     <!-- insert photonfocus_camera -->
-    <xacro:photonfocus_camera camera_name="$(arg camera_name)" parent="$(arg robot_name)_link_ee">
+    <xacro:photonfocus_camera camera_name="$(arg camera_name)" parent="$(arg robot_name)_link_ee" robot_name="$(arg robot_name)">
     </xacro:photonfocus_camera>
 </robot>

File: photonfocus_camera_description/urdf/photonfocus_camera.xacro (robot description, xacro)
@@ -1,13 +1,19 @@
 <?xml version="1.0" ?>
 <robot name="photonfocus_camera" xmlns:xacro="http://www.ros.org/wiki/xacro">
-<xacro:include filename="$(find photonfocus_camera_description)/urdf/materials.xacro" />
-<xacro:include filename="$(find photonfocus_camera_description)/urdf/photonfocus_camera.trans" />
-<xacro:include filename="$(find photonfocus_camera_description)/urdf/photonfocus_camera.gazebo"/>
-<xacro:macro name="photonfocus_camera" params="parent camera_name">
-	<link name="base_link">
+  <xacro:macro name="photonfocus_camera" params="camera_name robot_name parent">
+	<xacro:include filename="$(find photonfocus_camera_description)/urdf/materials.xacro" />
+	<xacro:include filename="$(find photonfocus_camera_description)/urdf/photonfocus_camera.trans" />
+	<xacro:include filename="$(find photonfocus_camera_description)/urdf/photonfocus_camera.gazebo" />
+	<!--joint between {parent} and base_link-->
+        <joint name="${parent}_${camera_name}_joint" type="fixed">
+            <parent link="${parent}"/>
+            <child link="${camera_name}_base_link"/>
+            <origin xyz="0 0 0" rpy="0 0 1.57079632679"/>
+        </joint>
+	<link name="${camera_name}_base_link">
 	  <inertial>
-	    <origin rpy="0 0 0" xyz="1.7763568394002505e-17 3.552713678800501e-17 0.0046742040606025685"/>
-	    <mass value="0.20307198484404515"/>
-	    <inertia ixx="4.8e-05" ixy="0.0" ixz="0.0" iyy="4.8e-05" iyz="0.0" izz="9.4e-05"/>
+	    <origin rpy="0 0 0" xyz="0.0004526550759665437 0.0005013636920587692 0.01966691095028127"/>
+	    <mass value="0.40283012340707985"/>
+	    <inertia ixx="0.000188" ixy="-0.0" ixz="-5e-06" iyy="0.000191" iyz="-0.0" izz="0.000112"/>
 	  </inertial>
 	  <visual>
@@ -25,34 +31,14 @@
 	  </collision>
 	</link>
-	<link name="Component8_1_1_1_1">
+	<link name="${camera_name}_link_1_1">
 	  <inertial>
-	    <origin rpy="0 0 0" xyz="0.006675819379415325 -0.0009462499931954823 0.025261336246706647"/>
-	    <mass value="0.1997581385630358"/>
-	    <inertia ixx="4.8e-05" ixy="-0.0" ixz="-2e-06" iyy="5.1e-05" iyz="-0.0" izz="1.8e-05"/>
-	  </inertial>
-	  <visual>
-	    <origin rpy="0 0 0" xyz="0.005763 -0.000949 -0.009647"/>
-	    <geometry>
-	      <mesh filename="package://photonfocus_camera_description/meshes/Component8_1_1_1_1.stl" scale="0.001 0.001 0.001"/>
-	    </geometry>
-	    <material name="silver"/>
-	  </visual>
-	  <collision>
-	    <origin rpy="0 0 0" xyz="0.005763 -0.000949 -0.009647"/>
-	    <geometry>
-	      <mesh filename="package://photonfocus_camera_description/meshes/Component8_1_1_1_1.stl" scale="0.001 0.001 0.001"/>
-	    </geometry>
-	  </collision>
-	</link>
-	<link name="Component7_1_1_1_1">
-	  <inertial>
-	    <origin rpy="0 0 0" xyz="0.00576299999995598 -0.0009489999999999939 0.006999172477632563"/>
-	    <mass value="0.010061892950917101"/>
-	    <inertia ixx="0.0" ixy="0.0" ixz="-0.0" iyy="0.0" iyz="0.0" izz="0.0"/>
+	    <origin rpy="0 0 0" xyz="-0.0029521431378939584 -0.015030724993614833 0.04528035169041975"/>
+	    <mass value="0.5898731797531614"/>
+	    <inertia ixx="0.000316" ixy="4e-06" ixz="-5e-06" iyy="0.000327" iyz="1.2e-05" izz="0.000271"/>
 	  </inertial>
 	  <visual>
 	    <origin rpy="0 0 0" xyz="0.005763 -0.000949 -0.059647"/>
 	    <geometry>
-	      <mesh filename="package://photonfocus_camera_description/meshes/Component7_1_1_1_1.stl" scale="0.001 0.001 0.001"/>
+	      <mesh filename="package://photonfocus_camera_description/meshes/link_1_1.stl" scale="0.001 0.001 0.001"/>
 	    </geometry>
 	    <material name="silver"/>
@@ -61,78 +47,18 @@
 	    <origin rpy="0 0 0" xyz="0.005763 -0.000949 -0.059647"/>
 	    <geometry>
-	      <mesh filename="package://photonfocus_camera_description/meshes/Component7_1_1_1_1.stl" scale="0.001 0.001 0.001"/>
+	      <mesh filename="package://photonfocus_camera_description/meshes/link_1_1.stl" scale="0.001 0.001 0.001"/>
 	    </geometry>
 	  </collision>
 	</link>
-	<link name="Component6_1_1_1_1">
+	<link name="${camera_name}_camera_link_1">
 	  <inertial>
-	    <origin rpy="0 0 0" xyz="0.005761639433104251 -0.009116655198803872 0.0050873760786627475"/>
-	    <mass value="0.07190809365548972"/>
-	    <inertia ixx="8e-06" ixy="0.0" ixz="-0.0" iyy="6e-06" iyz="-0.0" izz="1.3e-05"/>
-	  </inertial>
-	  <visual>
-	    <origin rpy="0 0 0" xyz="0.005763 -0.000949 -0.074647"/>
-	    <geometry>
-	      <mesh filename="package://photonfocus_camera_description/meshes/Component6_1_1_1_1.stl" scale="0.001 0.001 0.001"/>
-	    </geometry>
-	    <material name="silver"/>
-	  </visual>
-	  <collision>
-	    <origin rpy="0 0 0" xyz="0.005763 -0.000949 -0.074647"/>
-	    <geometry>
-	      <mesh filename="package://photonfocus_camera_description/meshes/Component6_1_1_1_1.stl" scale="0.001 0.001 0.001"/>
-	    </geometry>
-	  </collision>
-	</link>
-	<link name="Component2_1_1_1_1">
-	  <inertial>
-	    <origin rpy="0 0 0" xyz="-0.0012599221198894494 -0.019570473272113073 0.014158631511927311"/>
-	    <mass value="0.1371138450645388"/>
-	    <inertia ixx="6.1e-05" ixy="3e-06" ixz="0.0" iyy="2.8e-05" iyz="-3e-06" izz="6.1e-05"/>
-	  </inertial>
-	  <visual>
-	    <origin rpy="0 0 0" xyz="-0.002737 -0.000949 -0.084647"/>
-	    <geometry>
-	      <mesh filename="package://photonfocus_camera_description/meshes/Component2_1_1_1_1.stl" scale="0.001 0.001 0.001"/>
-	    </geometry>
-	    <material name="silver"/>
-	  </visual>
-	  <collision>
-	    <origin rpy="0 0 0" xyz="-0.002737 -0.000949 -0.084647"/>
-	    <geometry>
-	      <mesh filename="package://photonfocus_camera_description/meshes/Component2_1_1_1_1.stl" scale="0.001 0.001 0.001"/>
-	    </geometry>
-	  </collision>
-	</link>
-	<link name="Component3_1_1_1_1">
-	  <inertial>
-	    <origin rpy="0 0 0" xyz="-0.017468336612135094 -0.03067971553276897 0.0131744579556861"/>
-	    <mass value="0.37244365260000467"/>
-	    <inertia ixx="0.000149" ixy="1e-06" ixz="-5e-05" iyy="0.000171" iyz="1e-06" izz="0.000158"/>
-	  </inertial>
-	  <visual>
-	    <origin rpy="0 0 0" xyz="-0.003122 -0.015981 -0.099947"/>
-	    <geometry>
-	      <mesh filename="package://photonfocus_camera_description/meshes/Component3_1_1_1_1.stl" scale="0.001 0.001 0.001"/>
-	    </geometry>
-	    <material name="silver"/>
-	  </visual>
-	  <collision>
-	    <origin rpy="0 0 0" xyz="-0.003122 -0.015981 -0.099947"/>
-	    <geometry>
-	      <mesh filename="package://photonfocus_camera_description/meshes/Component3_1_1_1_1.stl" scale="0.001 0.001 0.001"/>
-	    </geometry>
-	  </collision>
-	</link>
-	<link name="Component4_1_1_1_1">
-	  <inertial>
-	    <origin rpy="0 0 0" xyz="-0.0031593464532001414 -0.07800866004916104 -0.0003471545903905998"/>
-	    <mass value="0.4535330539476499"/>
-	    <inertia ixx="0.000157" ixy="-1e-06" ixz="0.0" iyy="9.2e-05" iyz="2e-06" izz="0.000157"/>
+	    <origin rpy="0 0 0" xyz="-0.003122152950603064 -0.036121615255736886 0.00045540214292298653"/>
+	    <mass value="0.7434193408324884"/>
+	    <inertia ixx="0.003099" ixy="2e-06" ixz="1e-06" iyy="0.000111" iyz="-1.5e-05" izz="0.003097"/>
 	  </inertial>
 	  <visual>
 	    <origin rpy="0 0 0" xyz="-0.003237 -0.120949 -0.099647"/>
 	    <geometry>
-	      <mesh filename="package://photonfocus_camera_description/meshes/Component4_1_1_1_1.stl" scale="0.001 0.001 0.001"/>
+	      <mesh filename="package://photonfocus_camera_description/meshes/camera_link_1.stl" scale="0.001 0.001 0.001"/>
 	    </geometry>
 	    <material name="silver"/>
@@ -141,68 +67,43 @@
 	    <origin rpy="0 0 0" xyz="-0.003237 -0.120949 -0.099647"/>
 	    <geometry>
-	      <mesh filename="package://photonfocus_camera_description/meshes/Component4_1_1_1_1.stl" scale="0.001 0.001 0.001"/>
+	      <mesh filename="package://photonfocus_camera_description/meshes/camera_link_1.stl" scale="0.001 0.001 0.001"/>
 	    </geometry>
 	  </collision>
 	</link>
-	<link name="Component5_1_1_1_1">
+	<link name="${camera_name}_virtual_link_1">
 	  <inertial>
-	    <origin rpy="0 0 0" xyz="-0.05872928812870342 0.14692321997662616 0.0013688335279802288"/>
-	    <mass value="0.29377075965242594"/>
-	    <inertia ixx="0.000983" ixy="-0.0" ixz="-0.0" iyy="2.2e-05" iyz="1.3e-05" izz="0.00098"/>
+	    <origin rpy="0 0 0" xyz="-2.475900625821536e-07 -4.246171297905832e-08 0.0002504340682378259"/>
+	    <mass value="0.00011097676048806616"/>
+	    <inertia ixx="0.0" ixy="0.0" ixz="0.0" iyy="0.0" iyz="-0.0" izz="0.0"/>
 	  </inertial>
 	  <visual>
-	    <origin rpy="0 0 0" xyz="-0.058737 -0.000949 -0.099647"/>
+	    <origin rpy="0 0 0" xyz="-1.4e-05 -0.224948 -0.106917"/>
 	    <geometry>
-	      <mesh filename="package://photonfocus_camera_description/meshes/Component5_1_1_1_1.stl" scale="0.001 0.001 0.001"/>
+	      <mesh filename="package://photonfocus_camera_description/meshes/virtual_link_1.stl" scale="0.001 0.001 0.001"/>
 	    </geometry>
 	    <material name="silver"/>
 	  </visual>
 	  <collision>
-	    <origin rpy="0 0 0" xyz="-0.058737 -0.000949 -0.099647"/>
+	    <origin rpy="0 0 0" xyz="-1.4e-05 -0.224948 -0.106917"/>
 	    <geometry>
-	      <mesh filename="package://photonfocus_camera_description/meshes/Component5_1_1_1_1.stl" scale="0.001 0.001 0.001"/>
+	      <mesh filename="package://photonfocus_camera_description/meshes/virtual_link_1.stl" scale="0.001 0.001 0.001"/>
 	    </geometry>
 	  </collision>
 	</link>
-	<joint name="base_joint" type="fixed">
-	  <origin rpy="0 0 0" xyz="0 0 0"/>
-	  <parent link="${parent}"/>
-	  <child link="base_link"/>
+	<joint name="${camera_name}_joint_1" type="fixed">
+	  <origin rpy="0 0 0" xyz="-0.005763 0.000949 0.059647"/>
+	  <parent link="${camera_name}_base_link"/>
+	  <child link="${camera_name}_link_1_1"/>
 	</joint>
-	<joint name="Rigid28" type="fixed">
-	  <origin rpy="0 0 0" xyz="-0.005763 0.000949 0.009647"/>
-	  <parent link="base_link"/>
-	  <child link="Component8_1_1_1_1"/>
+	<joint name="${camera_name}_joint_2" type="fixed">
+	  <origin rpy="0 0 0" xyz="0.009 0.12 0.04"/>
+	  <parent link="${camera_name}_link_1_1"/>
+	  <child link="${camera_name}_camera_link_1"/>
 	</joint>
-	<joint name="Rigid29" type="fixed">
-	  <origin rpy="0 0 0" xyz="0.0 0.0 0.05"/>
-	  <parent link="Component8_1_1_1_1"/>
-	  <child link="Component7_1_1_1_1"/>
+	<joint name="${camera_name}_joint_3" type="fixed">
+	  <origin rpy="0 0 0" xyz="-0.003223 0.103999 0.00727"/>
+	  <parent link="${camera_name}_camera_link_1"/>
+	  <child link="${camera_name}_virtual_link_1"/>
 	</joint>
-	<joint name="Rigid30" type="fixed">
-	  <origin rpy="0 0 0" xyz="0.0 0.0 0.015"/>
-	  <parent link="Component7_1_1_1_1"/>
-	  <child link="Component6_1_1_1_1"/>
-	</joint>
-	<joint name="Rigid31" type="fixed">
-	  <origin rpy="0 0 0" xyz="0.0085 0.0 0.01"/>
-	  <parent link="Component6_1_1_1_1"/>
-	  <child link="Component2_1_1_1_1"/>
-	</joint>
-	<joint name="Rigid32" type="fixed">
-	  <origin rpy="0 0 0" xyz="0.000385 0.015032 0.0153"/>
-	  <parent link="Component2_1_1_1_1"/>
-	  <child link="Component3_1_1_1_1"/>
-	</joint>
-	<joint name="Rigid33" type="fixed">
-	  <origin rpy="0 0 0" xyz="0.0005 0.12 0.015"/>
-	  <parent link="Component2_1_1_1_1"/>
-	  <child link="Component4_1_1_1_1"/>
-	</joint>
-	<joint name="Rigid34" type="fixed">
-	  <origin rpy="0 0 0" xyz="0.0555 -0.12 0.0"/>
-	  <parent link="Component4_1_1_1_1"/>
-	  <child link="Component5_1_1_1_1"/>
-	</joint>
-</xacro:macro>
+  </xacro:macro>
 </robot>
